Commit message: Task A.3 completed

File: nuturtle_description/urdf/turtlebot3_burger.urdf.xacro (robot description, xacro)
@@ -3,4 +3,12 @@
   <xacro:include filename="$(find nuturtle_description)/urdf/common_properties.xacro"/>
   <xacro:include filename="$(find nuturtle_description)/urdf/turtlebot3_burger.gazebo.xacro"/>
+  <xacro:property name="yaml_file" value="$(find nuturtle_description)/config/diff_params.yaml"/>
+  <xacro:property name="props" value="${xacro.load_yaml(yaml_file)['/**']['ros__parameters']}"/>
+  <xacro:property name="wheel_radius" value="${props['wheel_radius']}"/>
+  <xacro:property name="track_width" value="${props['track_width']}"/>
+  <xacro:property name="motor_cmd_max" value="${props['motor_cmd_max']}"/>
+  <xacro:property name="motor_cmd_per_rad_sec" value="${props['motor_cmd_per_rad_sec']}"/>
+  <xacro:property name="encoder_ticks_per_rad" value="${props['encoder_ticks_per_rad']}"/>
+  <xacro:property name="collision_radius" value="${props['collision_radius']}"/>
   <link name="base_footprint"/>
   <joint name="base_joint" type="fixed">
@@ -19,7 +27,14 @@
     <collision>
       <origin xyz="-0.032 0 0.070" rpy="0 0 0"/>
-      <geometry>
-        <box size="0.140 0.140 0.143"/>
-      </geometry>
+      <xacro:if value="${collision_radius &lt; 0}">
+        <geometry>
+          <box size="0.140 0.140 0.143"/>
+        </geometry>
+      </xacro:if>
+      <xacro:if value="${collision_radius &gt;= 0}">
+        <geometry>
+          <cylinder length="0.143" radius="${collision_radius}"/>
+        </geometry>
+      </xacro:if>
     </collision>
     <inertial>
@@ -48,5 +63,5 @@
       <origin xyz="0 0 0" rpy="0 0 0"/>
       <geometry>
-        <cylinder length="0.018" radius="0.033"/>
+        <cylinder length="0.018" radius="${wheel_radius}"/>
       </geometry>
     </collision>
@@ -76,5 +91,5 @@
       <origin xyz="0 0 0" rpy="0 0 0"/>
       <geometry>
-        <cylinder length="0.018" radius="0.033"/>
+        <cylinder length="0.018" radius="${wheel_radius}"/>
       </geometry>
     </collision>

Commit message: Able to pass color to xacro

File: nuturtle_description/urdf/turtlebot3_burger.urdf.xacro (robot description, xacro)
@@ -3,4 +3,6 @@
   <xacro:include filename="$(find nuturtle_description)/urdf/common_properties.xacro"/>
   <xacro:include filename="$(find nuturtle_description)/urdf/turtlebot3_burger.gazebo.xacro"/>
+  <xacro:arg name="color" default="purple"/>
+  <xacro:property name="color" value="$(arg color)"/>
   <xacro:property name="yaml_file" value="$(find nuturtle_description)/config/diff_params.yaml"/>
   <xacro:property name="props" value="${xacro.load_yaml(yaml_file)['/**']['ros__parameters']}"/>
@@ -11,4 +13,7 @@
   <xacro:property name="encoder_ticks_per_rad" value="${props['encoder_ticks_per_rad']}"/>
   <xacro:property name="collision_radius" value="${props['collision_radius']}"/>
+  <material name="purple">
+    <color rgba="0.3 0.16 0.52 1.0"/>
+  </material>
   <link name="base_footprint"/>
   <joint name="base_joint" type="fixed">
@@ -23,5 +28,5 @@
         <mesh filename="package://nuturtle_description/meshes/burger_base.stl" scale="0.001 0.001 0.001"/>
       </geometry>
-      <material name="light_black"/>
+      <material name="${color}"/>
     </visual>
     <collision>
